Commit message: adding ikfast solution for bravo 7

File: output/robot.urdf (robot description, URDF)
Before this commit: robot /home/lukic/Documents/test.urdf, 7 links, 6 joints
Links:
- removed link base_link
- removed link solid_12158
- removed link solid_12168
- removed link solid_12178
- removed link solid_12188
- removed link solid_12198
- removed link solid_12208
- added link bravo_1013_joint_link, mass 1.14; collision cylinder length=0.03 radius=0.0408; collision cylinder length=0.03 radius=0.046
- added link bravo_1019_end_link, mass 1.55; collision cylinder length=0.03 radius=0.046; collision cylinder length=0.1 radius=0.046
- added link bravo_1023_0_joint_link, mass 0.333; collision cylinder length=0.08 radius=0.0408; visual mesh filename=package://bravo_description/meshes/RS2-1023_0_end.stl
- added link bravo_1023_1_joint_link, mass 1.04; collision cylinder length=0.0056 radius=0.0408; collision cylinder length=0.12 radius=0.0408
- added link bravo_1026_0_joint_link, mass 1.14; collision cylinder length=0.08 radius=0.0408; visual mesh filename=package://bravo_description/meshes/RS2-1026_0_end.stl
- added link bravo_1026_1_joint_link, mass 1.03; collision cylinder length=0.0056 radius=0.0408; collision cylinder length=0.03 radius=0.0408
- added link bravo_base_link, mass 1.25; collision box size=0.05 0.08 0.06; collision box size=0.0725 0.1112 0.083
- added link bravo_push_rod, mass 0.1
- added link ee_link
Joints:
- removed joint A motor
- removed joint B motor
- removed joint C motor
- removed joint D motor
- removed joint E motor
- removed joint F motor
- added joint bravo_axis_a: type prismatic, parent bravo_1023_1_joint_link, child bravo_push_rod, origin xyz=-8.669411487068951e-07 0.008999999958245167 0.12560000008350966 rpy=-1.5707 -1.5706999999997038 0.0, axis 0. 0. 1., limit lower=0.0 upper=0.035 effort=1000.0 velocity=10.0
- added joint bravo_axis_b: type continuous, parent bravo_1023_0_joint_link, child bravo_1023_1_joint_link, origin xyz=0.0408 -1.326794896676365e-09 -0.09434999999999824 rpy=3.14159 -0.0 0.0, axis  0.  0. -1., limit effort=500.0 velocity=6.0
- added joint bravo_axis_c: type revolute, parent bravo_1026_1_joint_link, child bravo_1023_0_joint_link, origin xyz=-0.041999999999852135 1.1145077132081467e-07 0.0634 rpy=0.0 -0.0 3.14159, axis  0. -1.  0., limit lower=0.0 upper=3.14 effort=500.0 velocity=6.0
- added joint bravo_axis_d: type revolute, parent bravo_1026_0_joint_link, child bravo_1026_1_joint_link, origin xyz=0.0408 -1.326794896676365e-09 -0.09434999999999824 rpy=3.14159 -0.0 0.0, axis  0.  0. -1., limit lower=0.0 upper=6.2 effort=500.0 velocity=6.0
- added joint bravo_axis_e: type revolute, parent bravo_1013_joint_link, child bravo_1026_0_joint_link, origin xyz=0.0040000000018364235 7.477816037645589e-07 -0.29034999999915573 rpy=3.14159 -0.0 3.14159, axis  0. -1.  0., limit lower=0.0 upper=3.14 effort=500.0 velocity=6.0
- added joint bravo_axis_f: type revolute, parent bravo_1019_end_link, child bravo_1013_joint_link, origin xyz=0.046 0.0 0.0642 rpy=0.0 -0.0 0.0, axis  0. -1.  0., limit lower=0.0 upper=3.14 effort=500.0 velocity=6.0
- added joint bravo_axis_g: type revolute, parent bravo_base_link, child bravo_1019_end_link, origin xyz=0.0665 0.0 0.08 rpy=0.0 0.0 3.14159, axis  0.  0. -1., limit lower=0.0 upper=6.2 effort=500.0 velocity=6.0
- added joint ee_link_joint: type fixed, parent bravo_1023_1_joint_link, child ee_link, origin xyz=0 0 0.120 rpy=0 0 -1.5707
